File: eurorack-bus-board-horizontal/eurorack-bus-board-horizontal.kicad_pcb (KiCad board)
At the start: 2 copper layers, 273.1 x 15.2 mm, 13 parts, among them J1 Power IN/THRU, J10 Conn_02x08_Eurorack, J2 Conn_02x08_Eurorack, J3 Conn_02x08_Eurorack, J5 Conn_02x08_Eurorack, J6 Conn_02x08_Eurorack, J7 Conn_02x08_Eurorack, J8 Conn_02x08_Eurorack, J9 Conn_02x08_Eurorack

Commit message: add additional files
Parts:
- J1: value Power IN/THRU -> Power In
- J10, J2, J3, J5, J6, J7, J8, J9: value Conn_02x08_Eurorack -> Euro 16-Pin; footprint Connector_IDC:IDC-Header_2x08_P2.54mm_Horizontal -> footprints:IDC-Header_2x08_P2.54mm_Horizontal_Quadrat
- moved H1 0.92 mm to (346.2, 104.9)
- moved H2 0.72 mm to (79.5, 104.9)
- moved H3 0.51 mm to (161.3, 104.9)
- moved H4 0.51 mm to (252.7, 104.9)
Connections:
- J10 pad 13: Net-(J10-Pad13) -> unconnected-(J10-Pad13)
- J10 pad 15: Net-(J10-Pad15) -> unconnected-(J10-Pad15)
- J2 pad 14: Net-(J2-Pad14) -> unconnected-(J2-Pad14)
- J2 pad 16: Net-(J2-Pad16) -> unconnected-(J2-Pad16)
- J3 pad 13: Net-(J2-Pad14) -> unconnected-(J3-Pad13)
- J3 pad 14: Net-(J3-Pad14) -> unconnected-(J3-Pad14)
- J3 pad 15: Net-(J2-Pad16) -> unconnected-(J3-Pad15)
- J3 pad 16: Net-(J3-Pad16) -> unconnected-(J3-Pad16)
- J5 pad 13: Net-(J3-Pad14) -> unconnected-(J5-Pad13)
- J5 pad 14: Net-(J5-Pad14) -> unconnected-(J5-Pad14)
- J5 pad 15: Net-(J3-Pad16) -> unconnected-(J5-Pad15)
- J5 pad 16: Net-(J5-Pad16) -> unconnected-(J5-Pad16)
- J6 pad 13: Net-(J5-Pad14) -> unconnected-(J6-Pad13)
- J6 pad 14: Net-(J6-Pad14) -> unconnected-(J6-Pad14)
- J6 pad 15: Net-(J5-Pad16) -> unconnected-(J6-Pad15)
- J6 pad 16: Net-(J6-Pad16) -> unconnected-(J6-Pad16)
- J7 pad 13: Net-(J6-Pad14) -> unconnected-(J7-Pad13)
- J7 pad 14: Net-(J7-Pad14) -> unconnected-(J7-Pad14)
- J7 pad 15: Net-(J6-Pad16) -> unconnected-(J7-Pad15)
- J7 pad 16: Net-(J7-Pad16) -> unconnected-(J7-Pad16)
- J8 pad 13: Net-(J7-Pad14) -> unconnected-(J8-Pad13)
- J8 pad 14: Net-(J8-Pad14) -> unconnected-(J8-Pad14)
- J8 pad 15: Net-(J7-Pad16) -> unconnected-(J8-Pad15)
- J8 pad 16: Net-(J8-Pad16) -> unconnected-(J8-Pad16)
- J9 pad 13: Net-(J8-Pad14) -> unconnected-(J9-Pad13)
- J9 pad 14: Net-(J10-Pad13) -> unconnected-(J9-Pad14)
- J9 pad 15: Net-(J8-Pad16) -> unconnected-(J9-Pad15)
- J9 pad 16: Net-(J10-Pad15) -> unconnected-(J9-Pad16)
Routing:
- net GND: vias 18 -> 20
- net -12V: vias 9 -> 8
Other:
- board text added: "- 8x 16-Pin Headers (no CV/Gate connections!) - Outer Copper Weight: 1 oz - Max rail current: 2A - Material: FR-4 (1.6 thickness)"
